File: PCB/half.kicad_sch (KiCad schematic)
At the start: 63 parts, among them J1 Battery Socket, SW3 SW_SPST, U1 Seeeduino Xiao nRF52840

Commit message: lfs here we go
Parts:
- added LED1, LED2, LED3, LED4, LED5, LED6: SK6812MINI-E, PCM_marbastlib-various:LED_6028R, symbol PCM_marbastlib-various:SK6812MINI-E
Connections:
- net GND: now also LED1.4 (VSS), LED2.4 (VSS), LED3.4 (VSS), LED4.4 (VSS), LED5.4 (VSS), LED6.4 (VSS)
- net LED: now reaches U1.17 (P0.09)
- net LED: now also LED1.3 (DIN)
- net VDD: now reaches U1.8 (5V)
- net VDD: now also LED1.1 (VDD), LED2.1 (VDD), LED3.1 (VDD), LED4.1 (VDD), LED5.1 (VDD), LED6.1 (VDD)
- new net: LED5.2 (DOUT), LED6.3 (DIN)
- new net: LED4.2 (DOUT), LED5.3 (DIN)
- new net: LED2.2 (DOUT), LED3.3 (DIN)
- new net: LED1.2 (DOUT), LED2.3 (DIN)
- new net: LED3.2 (DOUT), LED4.3 (DIN)
Other:
- note added: "LED's"
