File: PCB/right.kicad_sch (KiCad schematic)
At the start: 63 parts, among them J2 Battery Socket, SW4 SW_SPST, U2 Seeeduino Xiao nRF52840

Commit message: lfs here we go
Parts:
- added LED10, LED11, LED12, LED7, LED8, LED9: SK6812MINI-E, PCM_marbastlib-various:LED_6028R, symbol PCM_marbastlib-various:SK6812MINI-E
Connections:
- net GND: now also LED10.4 (VSS), LED11.4 (VSS), LED12.4 (VSS), LED7.4 (VSS), LED8.4 (VSS), LED9.4 (VSS)
- net LED: now reaches U2.17 (P0.09)
- net LED: now also LED7.3 (DIN)
- net VDD: now reaches U2.8 (5V)
- net VDD: now also LED10.1 (VDD), LED11.1 (VDD), LED12.1 (VDD), LED7.1 (VDD), LED8.1 (VDD), LED9.1 (VDD)
- new net: LED7.2 (DOUT), LED8.3 (DIN)
- new net: LED8.2 (DOUT), LED9.3 (DIN)
- new net: LED11.2 (DOUT), LED12.3 (DIN)
- new net: LED10.2 (DOUT), LED11.3 (DIN)
- new net: LED10.3 (DIN), LED9.2 (DOUT)
Other:
- note added: "LED's"
