File: PCB/split-keeb-v2.kicad_pcb (KiCad board)
At the start: 2 copper layers, 319.1 x 138.1 mm, 129 parts, among them J1 Battery Socket, J2 Battery Socket, SW3 SW_SPST, SW4 SW_SPST, U1 Seeeduino Xiao nRF52840, U2 Seeeduino Xiao nRF52840

Commit message: lfs here we go
Parts:
- removed BO1, BO2, BO3: break off, Mousebites:mouse-bite-5mm-slot
- added LED1: SK6812MINI-E, PCM_marbastlib-various:LED_6028R, B.Cu at (162.1, 102.2)
- added LED10: SK6812MINI-E, PCM_marbastlib-various:LED_6028R, B.Cu at (220.6, 120.7)
- added LED11: SK6812MINI-E, PCM_marbastlib-various:LED_6028R, B.Cu at (218.4, 111.5)
- added LED12: SK6812MINI-E, PCM_marbastlib-various:LED_6028R, B.Cu at (216.0, 102.0)
- added LED2: SK6812MINI-E, PCM_marbastlib-various:LED_6028R, B.Cu at (159.8, 111.5)
- added LED3: SK6812MINI-E, PCM_marbastlib-various:LED_6028R, B.Cu at (157.6, 120.7)
- added LED4: SK6812MINI-E, PCM_marbastlib-various:LED_6028R, B.Cu at (166.4, 122.9)
- added LED5: SK6812MINI-E, PCM_marbastlib-various:LED_6028R, B.Cu at (168.6, 113.6)
- added LED6: SK6812MINI-E, PCM_marbastlib-various:LED_6028R, B.Cu at (170.8, 104.3)
- added LED7: SK6812MINI-E, PCM_marbastlib-various:LED_6028R, B.Cu at (207.3, 104.3)
- added LED8: SK6812MINI-E, PCM_marbastlib-various:LED_6028R, B.Cu at (209.6, 113.6)
- added LED9: SK6812MINI-E, PCM_marbastlib-various:LED_6028R, B.Cu at (211.8, 122.9)
- D1, D10, D11, D12, D13, D14, D15, D16, D17, D18, D19, D2, D20, D21, D22, D23, D24, D25, D26, D27, D28, D29, D3, D30, D31, D32, D33, D34, D35, D36, D37, D38, D39, D4, D40, D41, D42, D43, D44, D45, D46, D47, D48, D49, D5, D50, D51, D52, D53, D54, D6, D7, D8, D9: footprint Diode_SMD:D_SOD-123 -> BAGEL-MISC:D_SOD-1n4148W-TP
- J1, J2: footprint PCM_marbastlib-various:CON_JST_ACH_BM02B -> PCM_SparkFun-Connector:JST_1x02_P2.0mm_Horizontal_PTH
- moved J2 344.1 mm to (216.7, 71.0), turned to 90 degrees
- moved H2 344.1 mm to (226.2, 133.8)
- moved R4 341.6 mm to (221.5, 69.5)
- moved R3 341.0 mm to (223.8, 69.5)
- moved H1 338.6 mm to (222.5, 89.5)
- moved CH30 335.4 mm to (272.9, 41.4)
- moved CH33 335.4 mm to (340.1, 57.1)
- moved CH36 335.4 mm to (274.9, 60.3)
- moved CH39 335.4 mm to (340.1, 76.2)
- moved CH41 335.4 mm to (256.8, 86.9)
- moved CH43 335.4 mm to (299.8, 81.5)
- moved CH45 335.4 mm to (340.1, 95.2)
- moved CH51 335.4 mm to (340.1, 114.3)
- moved D39 335.4 mm to (279.4, 103.2)
- moved D40 335.4 mm to (297.5, 48.5)
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Connections:
- U1 pad 17: unconnected-(U1-P0.09-Pad17) -> /left/LED
- U1 pad 8: unconnected-(U1-5V-Pad8) -> VDD
- U2 pad 17: unconnected-(U2-P0.09-Pad17) -> /right/LED
- U2 pad 8: unconnected-(U2-5V-Pad8) -> VDD
Routing:
- net VDD: track 0.00 -> 273.3 mm, vias 0 -> 1
- net GND: track 91.8 -> 277.6 mm, vias 0 -> 1
- net /left/LED: track 0.00 -> 38.6 mm
- net /right/LED: track 0.00 -> 37.9 mm
- net Net-(SW3-B): track 55.7 -> 33.7 mm
- net Net-(D41-A): track 0.00 -> 12.2 mm
- net Net-(LED10-DIN): track 0.00 -> 11.4 mm
- net /right/ROW4: track 132.2 -> 142.7 mm
- net Net-(LED3-DOUT): track 0.00 -> 10.2 mm
- net /left/ROW4: track 144.5 -> 149.8 mm
- net Net-(LED4-DOUT): track 0.00 -> 4.61 mm
- net Net-(LED5-DOUT): track 0.00 -> 4.61 mm
- net Net-(LED2-DOUT): track 0.00 -> 4.61 mm
- net Net-(LED1-DOUT): track 0.00 -> 4.61 mm
- net Net-(LED11-DOUT): track 0.00 -> 4.56 mm
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Other:
- board size 319.1 x 138.1 mm -> 330.5 x 136.5 mm
